Commit message: set toolframe offset to 7.5 cm instead of 11

File: katana_description/urdf/katana_450_6m180_simple.urdf.xacro (robot description, xacro)
@@ -11,5 +11,5 @@
   <property name="link4_length" value="0.1473" />
   <property name="link5_length" value="0.1505" />
-  <property name="tool_frame_offset" value="0.11" />
+  <property name="tool_frame_offset" value="0.075" />
   <!-- All inertial values (mass, center of mass and inertia tensor) have been
   calculated from the meshes using MeshLab -->
@@ -395,5 +395,5 @@
 		    <!-- The fake geometry here is only present to work around https://github.com/ros-planning/moveit_core/issues/158 -->
 		    <visual>
-		      <origin rpy="0 0 0" xyz="0 0 -0.075"/>
+		      <origin rpy="0 0 0" xyz="0 0 -${tool_frame_offset}"/>
 		      <geometry>
 			<box size="0.01 0.01 0.01"/>
@@ -402,5 +402,5 @@
 		    </visual>
 		    <collision>
-		      <origin rpy="0 0 0" xyz="0 0 -0.075"/>
+		      <origin rpy="0 0 0" xyz="0 0 -${tool_frame_offset}"/>
 		      <geometry>
 			<box size="0.01 0.01 0.01"/>
