Commit message: tuned down second joint velocity, regenerated urdf

File: katana_description/urdf/katana_450_6m180_simple.urdf (robot description, URDF)
Before this commit: robot katana_450_6m180, 11 links, 10 joints
Joints:
- joint katana_gripper_tool_agni_frame_joint: origin xyz=0 0 -0.11 rpy=0 3.14159265359 0 -> xyz=0 0 -0.075 rpy=0 3.14159265359 0
- joint katana_gripper_tool_frame_joint: origin xyz=0 0 -0.11 rpy=0 1.57079632679 0 -> xyz=0 0 -0.075 rpy=0 1.57079632679 0
- joint katana_motor1_pan_joint: limit lower=-3.0229511 upper=3.0123429 effort=1.5 velocity=2.208932 -> lower=-3.0229511 upper=3.0123429 effort=1.5 velocity=1.190799
- joint katana_motor2_lift_joint: limit lower=-2.6012933 upper=2.1639407 effort=0.6 velocity=1.190799 -> lower=-2.6012933 upper=2.1639407 effort=0.6 velocity=1.0
- joint katana_motor5_wrist_roll_joint: limit lower=-2.29926262 upper=3.016518 effort=0.01 velocity=2.208932 -> lower=-2.9926262 upper=3.016518 effort=0.01 velocity=2.208932

File: katana_description/urdf/katana_450_6m180_simple.urdf.xacro (robot description, xacro)
@@ -85,5 +85,5 @@
 	<origin xyz="0 0 0" rpy="${M_PI/2} 0 0"/>
 	<axis xyz="0 0 1"/>
-	<limit effort="0.6" lower="-2.6012933" upper="2.1639407"  velocity="1.190799"/>
+	<limit effort="0.6" lower="-2.6012933" upper="2.1639407"  velocity="1.0"/>
       </joint>
       <link name="katana_motor2_lift_link">
